File: hardware/kicad/EngModem_Modular_Routed_Rev5.kicad_sch (KiCad schematic)
At the start: 47 parts, among them J1 VFD, J10 ESP-ENABLE, J11 Micro_SD_Card, J12 DB9, J3 DC_PWR_HEADER, J4 MAX-ENCFG, J5 MAX-SHDN, J6 USB, J7 EXP, J8 MAX-MBAUD, J9 ESP-BOOT, U1 MAX3237EIPWR, U2 ESP32-S3-WROOM-1U, U3 LM7805S2/TR, U4 74HCT245, U5 LD1086D2T33TR

Commit message: Update the schematic: U4 symbol/value to CD74HCT640M
Adds a CD74HCT640M symbol to the RetroWiFiModem library (a sibling of the
existing 74HCT245 derived symbol, both extend the same base 74LS245A
graphic - the two parts are pin/pinout-identical, only the buffer
direction differs) and repoints U4's schematic instance at it, updating
both the live lib_id and the schematic's embedded lib_symbols cache.

Validated before committing: ERC produces the identical 32 violations
before and after (same types/descriptions, nothing new), and a netlist
export confirms U4's pin-to-net map is byte-identical - the fab data is
unaffected, only the part's identity in the design files changed.

Co-Authored-By: Claude Sonnet 5 <noreply@anthropic.com>
Parts:
- U4: value 74HCT245 -> CD74HCT640M; symbol RetroWiFiModem:74HCT245 -> RetroWiFiModem:CD74HCT640M
Changed lines of the file:
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@@
 	)
 	(symbol
-		(lib_id "RetroWiFiModem:74HCT245")
+		(lib_id "RetroWiFiModem:CD74HCT640M")
 		(at 81.28 71.12 0)
 		(unit 1)
@@
 			)
 		)
-		(property "Value" "74HCT245"
+		(property "Value" "CD74HCT640M"
 			(at 83.4233 54.61 0)
 			(show_name no)
